Commit message: child -> parent and add orientation initialization

File: robot.urdf (robot description, URDF)
Before this commit: robot my_first, 8 links, 7 joints
Links:
- added link connector_other_link; visual sphere radius=0.1
- added link other_link; visual cylinder length=0.5 radius=0.1
- link first_link: geometry visual cylinder length=2.0 radius=0.1
Joints:
- removed joint end_base_link
- added joint end_other_link: type continuous, parent connector_base_link, child other_link, origin xyz=0 0 0.1 rpy=1.5 0 0
- added joint end_third_link: type continuous, parent connector_second_link, child third_link, origin xyz=0 0 0.1 rpy=0 0 0
- added joint other_rigidity: type fixed, parent other_link, child connector_other_link, origin xyz=0 0 0.5
- joint end_first_link: child second_link -> first_link; origin xyz=0 0 0.1 -> xyz=0 0 0.1 rpy=0 0 0; parent connector_first_link -> connector_base_link
- joint end_second_link: child third_link -> second_link; origin xyz=0 0 0.1 -> xyz=0 0 0.1 rpy=0 0 0; parent connector_second_link -> connector_first_link
- joint first_rigidity: origin xyz=0 0 1.0 -> xyz=0 0 2.0

File: robot.xacro (robot description, xacro)
@@ -1,5 +1,15 @@
 <?xml version="1.0"?>
 <robot xmlns:xacro="http://www.ros.org/wiki/xacro" name="my_first">
-    <xacro:macro name="link" params="name size color child">
+    <xacro:macro
+        name="link"
+        params="name size color parent:='none' orientation:='0 0 0'"
+    >
+        <xacro:if value="${parent != 'none'}">
+            <joint name="end_${name}_link" type="continuous">
+                <parent link="connector_${parent}_link"/>
+                <child link="${name}_link"/>
+                <origin rpy="${orientation}" xyz="0 0 ${width}"/>
+            </joint>
+        </xacro:if>
         <link name="${name}_link">
             <visual>
@@ -7,5 +17,5 @@
                     <cylinder length="${size}" radius="${width}"/>
                 </geometry>
-                <origin rpy="0 0 0" xyz="0 0 ${size/2.}"/>
+                <origin rpy="0 0 0"  xyz="0 0 ${size/2.}"/>
                 <material name="${color}"/>
             </visual>
@@ -25,11 +35,4 @@
             </visual>
         </link>
-        <xacro:if value="${child != 'none'}">
-            <joint name="end_${name}_link" type="continuous">
-                <parent link="connector_${name}_link"/>
-                <child link="${child}_link"/>
-                <origin xyz="0 0 ${width}"/>
-            </joint>
-        </xacro:if>
     </xacro:macro>
     <material name="black">
@@ -40,7 +43,14 @@
     </material>
     <xacro:property name="width" value="0.1" />
-    <xacro:link name="base"   child="first"  size="0.6" color="white"/>
-    <xacro:link name="first"  child="second" size="1."  color="black"/>
-    <xacro:link name="second" child="third"  size="0.6" color="white"/>
-    <xacro:link name="third"  child="none"   size="0.6" color="black"/>
+    <xacro:link name="base"
+                size="0.6" color="white"/>
+    <xacro:link name="first"  parent="base"
+                size="2."  color="black"/>
+    <xacro:link name="other" parent="base"
+                orientation="1.5 0 0"
+                size="0.5"  color="black"/>
+    <xacro:link name="second" parent="first"
+                size="0.6" color="white"/>
+    <xacro:link name="third"  parent="second"
+                size="0.6" color="black"/>
 </robot>

Commit message: correct kinematic to enable rotation

File: robot.urdf (robot description, URDF)
Before this commit: robot my_first, 10 links, 9 joints
Links:
- link first_link: geometry visual cylinder length=0.9 radius=0.1
Joints:
- joint end_first_link: origin xyz=0 0 0.1 rpy=0 0 0 -> xyz=0 0 0 rpy=-1. 0 0
- joint end_other_link: origin xyz=0 0 0.1 rpy=1.5 0 0 -> xyz=0 0 0 rpy=1. 0 0
- joint end_second_link: origin xyz=0 0 0.1 rpy=0 0 0 -> xyz=0 0 0 rpy=0. 1.5 0
- joint end_third_link: origin xyz=0 0 0.1 rpy=0 0 0 -> xyz=0 0 0 rpy=0. 1.5 0
- joint first_rigidity: origin xyz=0 0 2.0 -> xyz=0 0 0.9

File: robot.xacro (robot description, xacro)
@@ -9,5 +9,5 @@
                 <parent link="connector_${parent}_link"/>
                 <child link="${name}_link"/>
-                <origin rpy="${orientation}" xyz="0 0 ${width}"/>
+                <origin rpy="${orientation}" xyz="0 0 0"/>
             </joint>
         </xacro:if>
@@ -17,5 +17,5 @@
                     <cylinder length="${size}" radius="${width}"/>
                 </geometry>
-                <origin rpy="0 0 0"  xyz="0 0 ${size/2.}"/>
+                <origin rpy="0 0 0"  xyz="0 0 ${size/2.+width}"/>
                 <material name="${color}"/>
             </visual>
@@ -24,5 +24,5 @@
             <parent link="${name}_link"/>
             <child link="connector_${name}_link"/>
-            <origin xyz="0 0 ${size}"/>
+            <origin xyz="0 0 ${size+width}"/>
         </joint>
         <link name="connector_${name}_link">
@@ -46,11 +46,14 @@
                 size="0.6" color="white"/>
     <xacro:link name="first"  parent="base"
-                size="2."  color="black"/>
+                orientation="-1. 0 0"
+                size="0.9"  color="black"/>
     <xacro:link name="other" parent="base"
-                orientation="1.5 0 0"
+                orientation="1. 0 0"
                 size="0.5"  color="black"/>
     <xacro:link name="second" parent="first"
+                orientation="0. 1.5 0"
                 size="0.6" color="white"/>
     <xacro:link name="third"  parent="second"
+                orientation="0. 1.5 0"
                 size="0.6" color="black"/>
 </robot>

Commit message: adding collision

File: robot.urdf (robot description, URDF)
Before this commit: robot my_first, 10 links, 9 joints
Links:
- link base_link: geometry collision cylinder length=0.6 radius=0.1; visual cylinder length=0.6 radius=0.1
- link connector_base_link: geometry collision sphere radius=0.1; visual sphere radius=0.1
- link connector_first_link: geometry collision sphere radius=0.1; visual sphere radius=0.1
- link connector_other_link: geometry collision sphere radius=0.1; visual sphere radius=0.1
- link connector_second_link: geometry collision sphere radius=0.1; visual sphere radius=0.1
- link connector_third_link: geometry collision sphere radius=0.1; visual sphere radius=0.1
- link first_link: geometry collision cylinder length=0.9 radius=0.1; visual cylinder length=0.9 radius=0.1
- link other_link: geometry collision cylinder length=0.5 radius=0.1; visual cylinder length=0.5 radius=0.1
- link second_link: geometry collision cylinder length=0.6 radius=0.1; visual cylinder length=0.6 radius=0.1
- link third_link: geometry collision cylinder length=0.6 radius=0.1; visual cylinder length=0.6 radius=0.1
Joints:
- joint base_rigidity: origin xyz=0 0 0.6 -> xyz=0 0 0.7
- joint end_second_link: origin xyz=0 0 0 rpy=0. 1.5 0 -> xyz=0 0 0 rpy=0. 3.14 0
- joint first_rigidity: origin xyz=0 0 0.9 -> xyz=0 0 1.0
- joint other_rigidity: origin xyz=0 0 0.5 -> xyz=0 0 0.6
- joint second_rigidity: origin xyz=0 0 0.6 -> xyz=0 0 0.7
- joint third_rigidity: origin xyz=0 0 0.6 -> xyz=0 0 0.7

File: robot.xacro (robot description, xacro)
@@ -20,4 +20,10 @@
                 <material name="${color}"/>
             </visual>
+            <collision>
+                <geometry>
+                    <cylinder length="${size}" radius="${width}"/>
+                </geometry>
+                <origin rpy="0 0 0"  xyz="0 0 ${size/2.+width}"/>
+            </collision>
         </link>
         <joint name="${name}_rigidity" type="fixed">
@@ -34,4 +40,10 @@
                 <material name="${color}"/>
             </visual>
+            <collision>
+                <geometry>
+                    <sphere radius="${width}"/>
+                </geometry>
+                <origin rpy="0 0 0" xyz="0 0 0"/>
+            </collision>
         </link>
     </xacro:macro>

Commit message: adding fake inertia

File: robot.urdf (robot description, URDF)
Before this commit: robot my_first, 10 links, 9 joints
Links:
- link connector_first_link: mass None -> 10
- link connector_other_link: mass None -> 10
- link connector_second_link: mass None -> 10
- link connector_third_link: mass None -> 10
- link first_link: mass None -> 10
- link other_link: mass None -> 10
- link second_link: mass None -> 10
- link third_link: mass None -> 10
Joints:
- joint end_second_link: origin xyz=0 0 0 rpy=0. 3.14 0 -> xyz=0 0 0 rpy=0. 1.5 0

File: robot.xacro (robot description, xacro)
@@ -26,4 +26,11 @@
                 <origin rpy="0 0 0"  xyz="0 0 ${size/2.+width}"/>
             </collision>
+            <xacro:if value="${parent != 'none'}">
+                <inertial>
+                    <mass value="10"/>
+                    <inertia ixx="0.4" ixy="0.0" ixz="0.0"
+                             iyy="0.4" iyz="0.0" izz="0.2"/>
+                </inertial>
+            </xacro:if>
         </link>
         <joint name="${name}_rigidity" type="fixed">
@@ -46,4 +53,11 @@
                 <origin rpy="0 0 0" xyz="0 0 0"/>
             </collision>
+            <xacro:if value="${parent != 'none'}">
+                <inertial>
+                    <mass value="10"/>
+                    <inertia ixx="0.4" ixy="0.0" ixz="0.0"
+                             iyy="0.4" iyz="0.0" izz="0.2"/>
+                </inertial>
+            </xacro:if>
         </link>
     </xacro:macro>
