Commit message: refactoring

File: urdf/robot.urdf (robot description, URDF)
Before this commit: robot my_first, 10 links, 9 joints
Links:
- link base_link: geometry collision cylinder length=0.6 radius=0.07; visual cylinder length=0.6 radius=0.07
- link connector_base_link: geometry collision sphere radius=0.07; visual sphere radius=0.07
- link connector_first_link: geometry collision sphere radius=0.07; visual sphere radius=0.07
- link connector_other_link: geometry collision sphere radius=0.07; visual sphere radius=0.07
- link connector_second_link: geometry collision sphere radius=0.07; visual sphere radius=0.07
- link connector_third_link: geometry collision sphere radius=0.07; visual sphere radius=0.07
- link first_link: geometry collision cylinder length=0.9 radius=0.07; visual cylinder length=0.9 radius=0.07
- link other_link: geometry collision cylinder length=0.5 radius=0.07; visual cylinder length=0.5 radius=0.07
- link second_link: geometry collision cylinder length=0.6 radius=0.07; visual cylinder length=0.6 radius=0.07
- link third_link: geometry collision cylinder length=0.6 radius=0.07; visual cylinder length=0.6 radius=0.07
Joints:
- joint base_rigidity: origin xyz=0 0 0.7 -> xyz=0 0 0.6699999999999999
- joint first_rigidity: origin xyz=0 0 1.0 -> xyz=0 0 0.97
- joint other_rigidity: origin xyz=0 0 0.6 -> xyz=0 0 0.5700000000000001
- joint second_rigidity: origin xyz=0 0 0.7 -> xyz=0 0 0.6699999999999999
- joint third_rigidity: origin xyz=0 0 0.7 -> xyz=0 0 0.6699999999999999

File: urdf/robot.xacro (robot description, xacro)
@@ -68,5 +68,5 @@
         <color rgba="1 1 1 1"/>
     </material>
-    <xacro:property name="width" value="0.1" />
+    <xacro:property name="width" value="0.07" />
     <xacro:link name="base"
                 size="0.6" color="white"/>
