Commit message: connect to gazebo

File: urdf/robot.xacro (robot description, xacro)
@@ -26,11 +26,12 @@
                 <origin rpy="0 0 0"  xyz="0 0 ${size/2.+width}"/>
             </collision>
-            <xacro:if value="${parent != 'none'}">
-                <inertial>
-                    <mass value="10"/>
-                    <inertia ixx="0.4" ixy="0.0" ixz="0.0"
-                             iyy="0.4" iyz="0.0" izz="0.2"/>
-                </inertial>
-            </xacro:if>
+            <!-- For gazebo, every link must have inertial -->
+            <!--<xacro:if value="${parent != 'none'}">-->
+            <inertial>
+                <mass value="10"/>
+                <inertia ixx="0.4" ixy="0.0" ixz="0.0"
+                         iyy="0.4" iyz="0.0" izz="0.2"/>
+            </inertial>
+            <!--</xacro:if>-->
         </link>
         <joint name="${name}_rigidity" type="fixed">
@@ -53,11 +54,12 @@
                 <origin rpy="0 0 0" xyz="0 0 0"/>
             </collision>
-            <xacro:if value="${parent != 'none'}">
-                <inertial>
-                    <mass value="10"/>
-                    <inertia ixx="0.4" ixy="0.0" ixz="0.0"
-                             iyy="0.4" iyz="0.0" izz="0.2"/>
-                </inertial>
-            </xacro:if>
+            <!--<xacro:if value="${parent != 'none'}">-->
+            <inertial>
+                <mass value="10"/>
+                <inertia ixx="0.4" ixy="0.0" ixz="0.0"
+                                   iyy="0.4" iyz="0.0"
+                                             izz="0.2"/>
+            </inertial>
+            <!--</xacro:if>-->
         </link>
     </xacro:macro>
@@ -69,4 +71,10 @@
     </material>
     <xacro:property name="width" value="0.07" />
+    <!-- Used for fixing robot to Gazebo 'base_link' -->
+    <link name="world"/>
+    <joint name="fixed" type="fixed">
+        <parent link="world"/>
+        <child  link="base_link"/>
+    </joint>
     <xacro:link name="base"
                 size="0.6" color="white"/>

Commit message: improving gazebo integration

File: urdf/robot.xacro (robot description, xacro)
@@ -71,7 +71,7 @@
     </material>
     <xacro:property name="width" value="0.07" />
-    <!-- Used for fixing robot to Gazebo 'base_link' -->
+    <!-- root link must not have inertia -->
     <link name="world"/>
-    <joint name="fixed" type="fixed">
+    <joint name="base_to_world" type="fixed">
         <parent link="world"/>
         <child  link="base_link"/>
